File: coffee-can-radar.sch (KiCad schematic (older format))
At the start: 45 parts

Commit message: Fixed potentiometer symbols, power labels, added Op-Amp OSC1 connected to Ramp_out
Parts:
- removed R?: 10K, symbol Device:R
- removed R?: 2M, symbol Device:R
- removed R?: 50K, symbol Device:R
- removed U? (x2): Opamp_Dual_Generic, symbol Device:Opamp_Dual_Generic
- added BT1: 12V, symbol Device:Battery
- added BT2: 6V, symbol Device:Battery
- added C?: 1 nF, symbol Device:C
- added J1: Conn_Coaxial, symbol Connector:Conn_Coaxial
- added R? (x3): 47K, symbol Device:R
- added RV1, RV3: 2M, symbol Device:R_POT
- added RV2: 50K, symbol Device:R_POT
- added U3, U?: OPA1604, symbol Amplifier_Operational:OPA1604
- added U? (x3): Opamp_Quad_Generic, symbol Device:Opamp_Quad_Generic
- gave numbers to parts that had none: 40
Connections:
- wire segments 95 -> 118
- no-connect marks 0 -> 6
Other:
- moved on the sheet: D1, R1, R13, R2
